File: Mainboard/Mainboard.brd (EAGLE design)
At the start: 150 x 120 mm, 60 parts, among them IC1 TL072CD, IC2 LM386M-1_NOPB, J1 USB3076, J2 640455-5, J3 640455-3, J4 640455-4, J5 640455-4, J6 SJ-3523-SMT-TR, J7 640455-2, J8 929850-01-06-RB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

Commit message: # Mainboard updated IX: final version (sd card size checked)
# EQ/VU-Meter final version added
Parts:
- moved C10 5.00 mm to (146.7, 57.3)
- moved J1 5.00 mm to (153.6, 57.3)
- moved C20 3.50 mm to (4.00, 86.0)
- moved J8 3.50 mm to (4.00, 82.5)
Routing:
- net -5V: track 209.8 -> 229.8 mm
- net GND: track 701.1 -> 714.6 mm, vias 784 -> 839
- net +5V: track 378.6 -> 383.6 mm
- net SD_DI: track 94.9 -> 98.4 mm
- net SD_CS: track 119.0 -> 122.5 mm
- net SD_CLK: track 66.2 -> 62.7 mm
- net +3V3: track 276.7 -> 273.2 mm
- net SD_DO: track 74.5 -> 71.0 mm
Other:
- board size 150 x 120 mm -> 160 x 120 mm
