File: EQ + VU-Meter/OLD/Equalizer_VUMeter.sch (EAGLE design)
At the start: 271 parts, among them IC1 TL072D, IC2 TL074D, IC3 TL074D, IC4 TL074D, IC5 TL072D, IC7 TL072D, J2 640455-4, T1 BC846A, T10 BC846A, T11 BC846A, T12 BC846A, T13 BC846A, T14 BC846A, T15 BC846A, T16 BC846A, T17 BC846A, T18 BC846A, T19 BC846A, T2 BC846A, T20 BC846A, T21 BC846A, T22 BC846A, T23 BC846A, T24 BC846A, T25 BC846A, T26 BC846A, T27 BC846A, T28 BC846A, T29 BC846A, T3 BC846A, T30 BC846A, T4 BC846A, T5 BC846A, T6 BC846A, T7 BC846A, T8 BC846A, T9 BC846A, U1 LM2611, U2 LMR62014

Commit message: # Mainboard updated
# Keyboard V2:

	# Bug fixed (lowest Pad not GND)
	# 1 more key (upper C)
	# PEACE sign corrected

# General cleanup
Parts:
- removed C10, C11, C12, C13, C27, C28, C29, C32, C39, C4, C8, C9: 100n, rcl:C-EUC0603
- removed C14, C40, C41, C42, C43, C44, C45, C46, C47, C48, C49, C50: 10u, rcl:C-EUC0603
- removed C5: 2.2 uF, rcl:C-EUC0603
- removed C7: 4.7 uF, rcl:C-EUC0603
- removed CCUK: 1 uF, rcl:C-EUC0603
- removed CF: 220 pF, rcl:C-EUC0603
- removed CFF: 330 pF, rcl:C-EUC0603
- removed CIN, COUT: 22 uF, rcl:C-EUC0603
- removed D14, D7: MMSZ5226B-7-F, MMSZ5226B-7-F:MMSZ5226B-7-F
- removed IC5, IC7: TL072D, linear:TL072D
- removed J2: 640455-4, 640455-4:640455-4
- removed L1, L2, L3: 10 uH, ASMCI-0603-100M-T:ASMCI-0603-100M-T
- removed R103, R104, R105: 0, rcl:R-EU_R0603
- removed R31: 68 K, rcl:R-EU_R0603
- removed R32: 51K, rcl:R-EU_R0603
- removed R35: 13.3K, rcl:R-EU_R0603
- removed R41: 3.3k, rcl:R-EU_R0603
- removed R42: 35K, rcl:R-EU_R0603
- removed RFB1: 29.4K, rcl:R-EU_R0603
- removed RFB2: 5.76K, rcl:R-EU_R0603
- removed U1: LM2611, LM2611BMFX_NOPB:LM2611BMFX/NOPB
- removed U2: LMR62014, LMR62014XMF_NOPB:LMR62014XMF/NOPB
- IC1: value TL072D -> TL074D; device linear:TL072D -> linear:TL074D; SPICEPREFIX (none) -> I
- IC2, IC3, IC4: SPICEPREFIX (none) -> I
- R26: value 0 -> 3.3k
- R27: value 0 -> 35K
Connections:
- removed net +7,5V: C45.2, C46.1, C47.1, C7.1, CF.1, CIN.1, D7.C, L2.1, R27.1, R31.2, U1.!SHDN, U1.VIN
- removed net -7,5V: C48.2, C49.1, C50.1, CFF.1, COUT.1, L3.2, R105.1, RFB1.1
- removed net IN2,1V: C38.2, J2.1
- removed net MAIN-5V: C14.2, C43.1, C44.1, J2.4, R103.1
- removed net N$100: IC3C.OUT, IC3D.+IN, R25.2
- removed net N$115: IC2C.OUT, IC2D.+IN, R6.2
- removed net N$126: CCUK.2, D14.A, L3.1
- removed net N$141: CCUK.1, L2.2, U1.SW
- removed net N$152: CFF.2, RFB1.2, RFB2.1, U1.NFB
- removed net N$16: C17.1, R29.2
- removed net N$18: C21.1, IC3B.OUT, R18.2, R19.1
- removed net N$181: IC2B.OUT, R3.1
- removed net N$183: IC4C.-IN, R41.2, R42.1
- removed net N$21: R32.1, U2.SHDN
- removed net N$22: CF.2, R31.1, R35.1, U2.FB
- removed net N$25: IC4C.OUT, IC4D.+IN, R42.2
- removed net N$48: C25.1, IC4B.OUT, R38.2, R41.1
- removed net N$74: D7.A, L1.2, U2.SW
- removed net PB5V: C40.2, C41.1, C42.1, C5.1, J2.2, L1.1, R104.2, R26.1, R26.2, R32.2, U2.VIN
- removed net V+: C27.1, C28.1, C29.1, C32.1, C39.1, C9.1, IC1P.V+, IC2P.V+, IC3P.V+, IC4P.V+, IC5P.V+, IC7P.V+, LD1.A, LD10.A, LD11.A, LD12.A, LD13.A, LD14.A, LD15.A, LD16.A, LD17.A, LD18.A, LD19.A, LD2.A, LD20.A, LD21.A, LD22.A, LD23.A, LD24.A, LD25.A, LD26.A, LD27.A, LD28.A, LD29.A, LD3.A, LD30.A, LD4.A, LD5.A, LD6.A, LD7.A, LD8.A, LD9.A, R104.1, R27.2
- removed net V-: C10.2, C11.2, C12.2, C13.2, C4.2, C8.2, IC1P.V-, IC2P.V-, IC3P.V-, IC4P.V-, IC5P.V-, IC7P.V-, R103.2, R105.2
- new net +8V: IC1P.V+, IC2P.V+, IC3P.V+, IC4P.V+, LD1.A, LD10.A, LD11.A, LD12.A, LD13.A, LD14.A, LD15.A, LD16.A, LD17.A, LD18.A, LD19.A, LD2.A, LD20.A, LD21.A, LD22.A, LD23.A, LD24.A, LD25.A, LD26.A, LD27.A, LD28.A, LD29.A, LD3.A, LD30.A, LD4.A, LD5.A, LD6.A, LD7.A, LD8.A, LD9.A
- new net -8V: IC1P.V-, IC2P.V-, IC3P.V-, IC4P.V-
- new net 3.3V: C38.2
- new net N$1: C2.1, C3.1
- new net N$14: IC3D.-IN, R26.2, R27.1
- new net N$6: C1.1, C6.1
- new net TP_OUT1: IC2C.OUT, R6.2
- new net TP_OUT2: IC3B.OUT, R25.2
- new net TP_OUT3: IC3D.OUT, R27.2
- net BP1_OUT: now also C17.1, IC2B.OUT, R29.2, R3.1; no longer IC2D.-IN, IC2D.OUT
- net BP2_OUT: now also C21.1, IC3A.OUT, R18.2, R19.1; no longer IC3D.-IN, IC3D.OUT
- net BP3_OUT: now also C25.1, IC4A.OUT, R26.1, R38.2; no longer IC4D.-IN, IC4D.OUT
- net GND: now also IC1C.+IN, IC1D.+IN, IC2D.+IN, IC3D.+IN; no longer C10.1, C11.1, C12.1, C13.1, C14.1, C27.2, C28.2, C29.2, C32.2, C39.2, C4.1, C40.1, C41.2, C42.2, C43.2, C44.2, C45.1, C46.2, C47.2, C48.1, C49.2, C5.2, C50.2, C7.2, C8.1, C9.2, CIN.2, COUT.2, D14.C, IC1A.+IN, IC4C.+IN, IC5B.+IN, IC7B.+IN, J2.3, R35.2, RFB2.2, U1.GND, U2.GND
- net HP_OUT: now also IC4B.OUT; no longer IC7B.OUT
- net N$10: now also IC1D.-IN; no longer IC1B.-IN
- net N$19: now also IC2D.-IN; no longer IC3A.-IN
- net N$2: no longer C1.1, C6.1
- net N$20: now also IC2D.OUT; no longer IC3A.OUT
- net N$24: now also IC3A.-IN; no longer IC3B.-IN
- net N$26: now also IC3C.OUT; no longer IC4A.OUT
- net N$28: now also IC3C.-IN; no longer IC4A.-IN
- net N$29: now also IC1B.-IN; no longer IC5B.-IN
- net N$3: now also IC1C.-IN; no longer IC1A.-IN
- net N$32: now also IC4A.-IN; no longer IC4B.-IN
- net N$34: now also IC4C.+IN; no longer IC7A.+IN
- net N$36: now also IC4C.-IN, IC4C.OUT; no longer IC7A.-IN, IC7A.OUT
- net N$39: now also IC4B.-IN; no longer IC7B.-IN
- net N$4: no longer C2.1, C3.1
- net N$42: now also IC1A.-IN, IC1A.OUT; no longer IC5A.-IN, IC5A.OUT
- net N$47: now also IC1A.+IN; no longer IC5A.+IN
- net N$5: now also IC1B.OUT; no longer IC5B.OUT
- net N$8: now also IC1C.OUT; no longer IC1A.OUT
- net N$9: now also IC3B.-IN; no longer IC3C.-IN
- net TP_OUT: now also IC1D.OUT; no longer IC1B.OUT
Other:
- moved on the sheet: C37, D104, D29, D30, D31, D32, D33, D34, IC1A, IC1B, IC2C, IC2D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

Commit message: Production data for ordering Mainboard, Keys, UI and EQ at JLCPCB
Parts:
- added C10, C11, C12, C13, C27, C28, C29, C32, C39, C4, C8, C9: 100n, rcl:C-EUC0603
- added C14, C40, C41, C42, C43, C44, C45, C46, C47, C48, C49, C50: 10u, rcl:C-EUC0603
- added C5: 2.2 uF, rcl:C-EUC0603
- added C7: 4.7 uF, rcl:C-EUC0603
- added CCUK: 1 uF, rcl:C-EUC0603
- added CF: 220 pF, rcl:C-EUC0603
- added CFF: 330 pF, rcl:C-EUC0603
- added CIN, COUT: 22 uF, rcl:C-EUC0603
- added D14, D7: MMSZ5226B-7-F, MMSZ5226B-7-F:MMSZ5226B-7-F
- added IC5, IC7: TL072D, linear:TL072D
- added J2: 640455-4, 640455-4:640455-4
- added L1, L2, L3: 10 uH, ASMCI-0603-100M-T:ASMCI-0603-100M-T
- added R103, R104, R105: 0, rcl:R-EU_R0603
- added R31: 68 K, rcl:R-EU_R0603
- added R32: 51K, rcl:R-EU_R0603
- added R35: 13.3K, rcl:R-EU_R0603
- added R41: 3.3k, rcl:R-EU_R0603
- added R42: 35K, rcl:R-EU_R0603
- added RFB1: 29.4K, rcl:R-EU_R0603
- added RFB2: 5.76K, rcl:R-EU_R0603
- added U1: LM2611, LM2611BMFX_NOPB:LM2611BMFX/NOPB
- added U2: LMR62014, LMR62014XMF_NOPB:LMR62014XMF/NOPB
- IC1: value TL074D -> TL072D; device linear:TL074D -> linear:TL072D; SPICEPREFIX I -> (none)
- IC2, IC3, IC4: SPICEPREFIX I -> (none)
- R26: value 3.3k -> 0
- R27: value 35K -> 0
Connections:
- removed net +8V: IC1P.V+, IC2P.V+, IC3P.V+, IC4P.V+, LD1.A, LD10.A, LD11.A, LD12.A, LD13.A, LD14.A, LD15.A, LD16.A, LD17.A, LD18.A, LD19.A, LD2.A, LD20.A, LD21.A, LD22.A, LD23.A, LD24.A, LD25.A, LD26.A, LD27.A, LD28.A, LD29.A, LD3.A, LD30.A, LD4.A, LD5.A, LD6.A, LD7.A, LD8.A, LD9.A
- removed net -8V: IC1P.V-, IC2P.V-, IC3P.V-, IC4P.V-
- removed net 3.3V: C38.2
- removed net N$1: C2.1, C3.1
- removed net N$14: IC3D.-IN, R26.2, R27.1
- removed net N$6: C1.1, C6.1
- removed net TP_OUT1: IC2C.OUT, R6.2
- removed net TP_OUT2: IC3B.OUT, R25.2
- removed net TP_OUT3: IC3D.OUT, R27.2
- new net +7,5V: C45.2, C46.1, C47.1, C7.1, CF.1, CIN.1, D7.C, L2.1, R27.1, R31.2, U1.!SHDN, U1.VIN
- new net -7,5V: C48.2, C49.1, C50.1, CFF.1, COUT.1, L3.2, R105.1, RFB1.1
- new net IN2,1V: C38.2, J2.1
- new net MAIN-5V: C14.2, C43.1, C44.1, J2.4, R103.1
- new net N$100: IC3C.OUT, IC3D.+IN, R25.2
- new net N$115: IC2C.OUT, IC2D.+IN, R6.2
- new net N$126: CCUK.2, D14.A, L3.1
- new net N$141: CCUK.1, L2.2, U1.SW
- new net N$152: CFF.2, RFB1.2, RFB2.1, U1.NFB
- new net N$16: C17.1, R29.2
- new net N$18: C21.1, IC3B.OUT, R18.2, R19.1
- new net N$181: IC2B.OUT, R3.1
- new net N$183: IC4C.-IN, R41.2, R42.1
- new net N$21: R32.1, U2.SHDN
- new net N$22: CF.2, R31.1, R35.1, U2.FB
- new net N$25: IC4C.OUT, IC4D.+IN, R42.2
- new net N$48: C25.1, IC4B.OUT, R38.2, R41.1
- new net N$74: D7.A, L1.2, U2.SW
- new net PB5V: C40.2, C41.1, C42.1, C5.1, J2.2, L1.1, R104.2, R26.1, R26.2, R32.2, U2.VIN
- new net V+: C27.1, C28.1, C29.1, C32.1, C39.1, C9.1, IC1P.V+, IC2P.V+, IC3P.V+, IC4P.V+, IC5P.V+, IC7P.V+, LD1.A, LD10.A, LD11.A, LD12.A, LD13.A, LD14.A, LD15.A, LD16.A, LD17.A, LD18.A, LD19.A, LD2.A, LD20.A, LD21.A, LD22.A, LD23.A, LD24.A, LD25.A, LD26.A, LD27.A, LD28.A, LD29.A, LD3.A, LD30.A, LD4.A, LD5.A, LD6.A, LD7.A, LD8.A, LD9.A, R104.1, R27.2
- new net V-: C10.2, C11.2, C12.2, C13.2, C4.2, C8.2, IC1P.V-, IC2P.V-, IC3P.V-, IC4P.V-, IC5P.V-, IC7P.V-, R103.2, R105.2
- net BP1_OUT: now also IC2D.-IN, IC2D.OUT; no longer C17.1, IC2B.OUT, R29.2, R3.1
- net BP2_OUT: now also IC3D.-IN, IC3D.OUT; no longer C21.1, IC3A.OUT, R18.2, R19.1
- net BP3_OUT: now also IC4D.-IN, IC4D.OUT; no longer C25.1, IC4A.OUT, R26.1, R38.2
- net GND: now also C10.1, C11.1, C12.1, C13.1, C14.1, C27.2, C28.2, C29.2, C32.2, C39.2, C4.1, C40.1, C41.2, C42.2, C43.2, C44.2, C45.1, C46.2, C47.2, C48.1, C49.2, C5.2, C50.2, C7.2, C8.1, C9.2, CIN.2, COUT.2, D14.C, IC1A.+IN, IC4C.+IN, IC5B.+IN, IC7B.+IN, J2.3, R35.2, RFB2.2, U1.GND, U2.GND; no longer IC1C.+IN, IC1D.+IN, IC2D.+IN, IC3D.+IN
- net HP_OUT: now also IC7B.OUT; no longer IC4B.OUT
- net N$10: now also IC1B.-IN; no longer IC1D.-IN
- net N$19: now also IC3A.-IN; no longer IC2D.-IN
- net N$2: now also C1.1, C6.1
- net N$20: now also IC3A.OUT; no longer IC2D.OUT
- net N$24: now also IC3B.-IN; no longer IC3A.-IN
- net N$26: now also IC4A.OUT; no longer IC3C.OUT
- net N$28: now also IC4A.-IN; no longer IC3C.-IN
- net N$29: now also IC5B.-IN; no longer IC1B.-IN
- net N$3: now also IC1A.-IN; no longer IC1C.-IN
- net N$32: now also IC4B.-IN; no longer IC4A.-IN
- net N$34: now also IC7A.+IN; no longer IC4C.+IN
- net N$36: now also IC7A.-IN, IC7A.OUT; no longer IC4C.-IN, IC4C.OUT
- net N$39: now also IC7B.-IN; no longer IC4B.-IN
- net N$4: now also C2.1, C3.1
- net N$42: now also IC5A.-IN, IC5A.OUT; no longer IC1A.-IN, IC1A.OUT
- net N$47: now also IC5A.+IN; no longer IC1A.+IN
- net N$5: now also IC5B.OUT; no longer IC1B.OUT
- net N$8: now also IC1A.OUT; no longer IC1C.OUT
- net N$9: now also IC3C.-IN; no longer IC3B.-IN
- net TP_OUT: now also IC1B.OUT; no longer IC1D.OUT
Other:
- moved on the sheet: C37, D104, D29, D30, D31, D32, D33, D34, IC1A, IC1B, IC2C, IC2D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
